File: M.2 Type 2242-XX-B/adf7021.sch (KiCad schematic (older format))
At the start: 47 parts, among them U1 M74VHC1GT04DFT1G, U2 AS193-73, U4 ADF7021BCPZ, X1 FT5HNBPK19.44-T1

Commit message: Add proper footprint to solder jumpers
Parts:
- renumbered U1 to U3
Changed lines of the file:
@@
 AR Path="/5CA93143/5DAD1866" Ref="U?"  Part="1"
 AR Path="/5DA4D1CA/5DAD1866" Ref="U?"  Part="1"
-AR Path="/5DA99182/5DAD1866" Ref="U1"  Part="1"
+AR Path="/5DA99182/5DAD1866" Ref="U3"  Part="1"
 AR Path="/5DC39AF2/5DAD1866" Ref="U?"  Part="1"
 AR Path="/5DC39DB3/5DAD1866" Ref="U?"  Part="1"
 AR Path="/5DC39F66/5DAD1866" Ref="U?"  Part="1"
-F 0 "U1" H 2050 1617 50  0000 C CNN
+F 0 "U3" H 2050 1617 50  0000 C CNN
 F 1 "M74VHC1GT04DFT1G" H 2050 1526 50  0000 C CNN
 F 2 "Package_TO_SOT_SMD:SOT-353_SC-70-5" H 2050 1250 50  0001 C CNN

Commit message: NOP Update
Parts:
- removed JP5: SolderJumper_2_Bridged, Jumper:SolderJumper-2_P1.3mm_Bridged_RoundedPad1.0x1.5mm, symbol Jumper:SolderJumper_2_Bridged
- C34, C35, C4: footprint (none) -> Capacitor_SMD:C_0603_1608Metric
- L4, L5, L6: footprint (none) -> Inductor_SMD:L_0603_1608Metric
Connections:
- net +3V3: now also C19.1, X1.4 (Vdd)
Changed lines of the file:
@@
 NOTE: This is to make it easy to hack\nif we need to test with seperate supply.
 $Comp
-L Jumper:SolderJumper_2_Bridged JP?
-U 1 1 5DAD1973
-P 7250 1000
-AR Path="/5CA93306/5DAD1973" Ref="JP?"  Part="1"
-AR Path="/5CA93143/5DAD1973" Ref="JP?"  Part="1"
-AR Path="/5DA4D1CA/5DAD1973" Ref="JP?"  Part="1"
-AR Path="/5DA99182/5DAD1973" Ref="JP5"  Part="1"
-AR Path="/5DC39AF2/5DAD1973" Ref="JP?"  Part="1"
-AR Path="/5DC39DB3/5DAD1973" Ref="JP?"  Part="1"
-AR Path="/5DC39F66/5DAD1973" Ref="JP?"  Part="1"
-F 0 "JP5" V 7204 1068 50  0000 L CNN
-F 1 "SolderJumper_2_Bridged" V 7295 1068 50  0000 L CNN
-F 2 "Jumper:SolderJumper-2_P1.3mm_Bridged_RoundedPad1.0x1.5mm" H 7250 1000 50  0001 C CNN
-F 3 "~" H 7250 1000 50  0001 C CNN
-	1    7250 1000
-	0    1    1    0
-$EndComp
-$Comp
 L power:GND #PWR?
 U 1 1 5DAD193A
@@
 L power:+3.3V #PWR?
 U 1 1 5DAD179E
-P 7250 850
+P 7250 1150
 AR Path="/5CA93306/5DAD179E" Ref="#PWR?"  Part="1"
 AR Path="/5CA93143/5DAD179E" Ref="#PWR?"  Part="1"
@@
 AR Path="/5DC39DB3/5DAD179E" Ref="#PWR?"  Part="1"
 AR Path="/5DC39F66/5DAD179E" Ref="#PWR?"  Part="1"
-F 0 "#PWR0118" H 7250 700 50  0001 C CNN
-F 1 "+3.3V" H 7265 1023 50  0000 C CNN
-F 2 "" H 7250 850 50  0001 C CNN
-F 3 "" H 7250 850 50  0001 C CNN
-	1    7250 850
+F 0 "#PWR0118" H 7250 1000 50  0001 C CNN
+F 1 "+3.3V" H 7265 1323 50  0000 C CNN
+F 2 "" H 7250 1150 50  0001 C CNN
+F 3 "" H 7250 1150 50  0001 C CNN
+	1    7250 1150
 	1    0    0    -1
 $EndComp
@@
 F 0 "L6" V 2490 4550 50  0000 C CNN
 F 1 "20nH" V 2399 4550 50  0000 C CNN
-F 2 "" H 2300 4550 50  0001 C CNN
+F 2 "Inductor_SMD:L_0603_1608Metric" H 2300 4550 50  0001 C CNN
 F 3 "~" H 2300 4550 50  0001 C CNN
 	1    2300 4550
@@
 F 0 "L5" V 1990 4550 50  0000 C CNN
 F 1 "22nH" V 1899 4550 50  0000 C CNN
-F 2 "" H 1800 4550 50  0001 C CNN
+F 2 "Inductor_SMD:L_0603_1608Metric" H 1800 4550 50  0001 C CNN
 F 3 "~" H 1800 4550 50  0001 C CNN
 	1    1800 4550
@@
 F 0 "C35" H 2665 4846 50  0000 L CNN
 F 1 "C" H 2665 4755 50  0000 L CNN
-F 2 "" H 2588 4650 50  0001 C CNN
+F 2 "Capacitor_SMD:C_0603_1608Metric" H 2588 4650 50  0001 C CNN
 F 3 "~" H 2550 4800 50  0001 C CNN
 	1    2550 4800
@@
 F 0 "C34" H 2165 4846 50  0000 L CNN
 F 1 "6.8pF" H 2165 4755 50  0000 L CNN
-F 2 "" H 2088 4650 50  0001 C CNN
+F 2 "Capacitor_SMD:C_0603_1608Metric" H 2088 4650 50  0001 C CNN
 F 3 "~" H 2050 4800 50  0001 C CNN
 	1    2050 4800
@@
 F 0 "C4" H 1665 4846 50  0000 L CNN
 F 1 "C" H 1665 4755 50  0000 L CNN
-F 2 "" H 1588 4650 50  0001 C CNN
+F 2 "Capacitor_SMD:C_0603_1608Metric" H 1588 4650 50  0001 C CNN
 F 3 "~" H 1550 4800 50  0001 C CNN
 	1    1550 4800
@@
 F 0 "L4" V 1490 4550 50  0000 C CNN
 F 1 "0R" V 1399 4550 50  0000 C CNN
-F 2 "" H 1300 4550 50  0001 C CNN
+F 2 "Inductor_SMD:L_0603_1608Metric" H 1300 4550 50  0001 C CNN
 F 3 "~" H 1300 4550 50  0001 C CNN
 	1    1300 4550

Commit message: Initial placement, I think we are going for the STM32F103 instead
The LQPF-100 is simply too big
Parts:
- C1: value 22uF -> 10uF; footprint Capacitor_SMD:C_1812_4532Metric -> Capacitor_SMD:C_0603_1608Metric
- C10, C11, C12, C13, C14, C15, C16, C17, C18, C19, C2, C20, C21, C22, C23, C3, C34, C35, C36, C4, C5, C6, C7, C8, C9: footprint Capacitor_SMD:C_0603_1608Metric -> Capacitor_SMD:C_0402_1005Metric
- R1, R2, R3, R4, R5, R6, R7, R8: footprint Resistor_SMD:R_0603_1608Metric -> Resistor_SMD:R_0402_1005Metric
Changed lines of the file:
@@
 AR Path="/5DC39F66/5DAD15C9" Ref="C?"  Part="1"
 F 0 "C1" H 1015 7096 50  0000 L CNN
-F 1 "22uF" H 1015 7005 50  0000 L CNN
-F 2 "Capacitor_SMD:C_1812_4532Metric" H 938 6900 50  0001 C CNN
+F 1 "10uF" H 1015 7005 50  0000 L CNN
+F 2 "Capacitor_SMD:C_0603_1608Metric" H 938 6900 50  0001 C CNN
 F 3 "~" H 900 7050 50  0001 C CNN
 F 4 "CAP CER 10UF 16V X7R 1812" H 900 7050 50  0001 C CNN "manf#"
@@
 F 0 "C8" H 3385 3346 50  0000 R CNN
 F 1 "220pF" H 3385 3255 50  0000 R CNN
-F 2 "Capacitor_SMD:C_0603_1608Metric" H 3538 3150 50  0001 C CNN
+F 2 "Capacitor_SMD:C_0402_1005Metric" H 3538 3150 50  0001 C CNN
 F 3 "~" H 3500 3300 50  0001 C CNN
 	1    3500 3300
@@
 F 0 "C6" H 3365 3346 50  0000 L CNN
 F 1 "10nF" H 3365 3255 50  0000 L CNN
-F 2 "Capacitor_SMD:C_0603_1608Metric" H 3288 3150 50  0001 C CNN
+F 2 "Capacitor_SMD:C_0402_1005Metric" H 3288 3150 50  0001 C CNN
 F 3 "~" H 3250 3300 50  0001 C CNN
 	1    3250 3300
@@
 F 0 "C3" V 1310 2250 50  0000 C CNN
 F 1 "100pF" V 1401 2250 50  0000 C CNN
-F 2 "Capacitor_SMD:C_0603_1608Metric" H 1188 2100 50  0001 C CNN
+F 2 "Capacitor_SMD:C_0402_1005Metric" H 1188 2100 50  0001 C CNN
 F 3 "~" H 1150 2250 50  0001 C CNN
 	1    1150 2250
@@
 F 0 "C2" V 898 2050 50  0000 C CNN
 F 1 "100pF" V 989 2050 50  0000 C CNN
-F 2 "Capacitor_SMD:C_0603_1608Metric" H 1188 1900 50  0001 C CNN
+F 2 "Capacitor_SMD:C_0402_1005Metric" H 1188 1900 50  0001 C CNN
 F 3 "~" H 1150 2050 50  0001 C CNN
 	1    1150 2050
@@
 F 0 "C5" V 2198 2150 50  0000 C CNN
 F 1 "100pF" V 2289 2150 50  0000 C CNN
-F 2 "Capacitor_SMD:C_0603_1608Metric" H 2488 2000 50  0001 C CNN
+F 2 "Capacitor_SMD:C_0402_1005Metric" H 2488 2000 50  0001 C CNN
 F 3 "~" H 2450 2150 50  0001 C CNN
 	1    2450 2150
@@
 F 0 "C19" H 7715 1446 50  0000 L CNN
 F 1 "10nF" H 7715 1355 50  0000 L CNN
-F 2 "Capacitor_SMD:C_0603_1608Metric" H 7638 1250 50  0001 C CNN
+F 2 "Capacitor_SMD:C_0402_1005Metric" H 7638 1250 50  0001 C CNN
 F 3 "~" H 7600 1400 50  0001 C CNN
 	1    7600 1400
@@
 F 0 "C10" V 4298 3050 50  0000 C CNN
 F 1 "100nF" V 4389 3050 50  0000 C CNN
-F 2 "Capacitor_SMD:C_0603_1608Metric" H 4588 2900 50  0001 C CNN
+F 2 "Capacitor_SMD:C_0402_1005Metric" H 4588 2900 50  0001 C CNN
 F 3 "~" H 4550 3050 50  0001 C CNN
 	1    4550 3050
@@
 F 0 "R2" V 4743 3050 50  0000 C CNN
 F 1 "3R9" V 4834 3050 50  0000 C CNN
-F 2 "Resistor_SMD:R_0603_1608Metric" V 4880 3050 50  0001 C CNN
+F 2 "Resistor_SMD:R_0402_1005Metric" V 4880 3050 50  0001 C CNN
 F 3 "~" H 4950 3050 50  0001 C CNN
 	1    4950 3050
@@
 F 0 "C21" H 8465 4746 50  0000 L CNN
 F 1 "100nF" H 8465 4655 50  0000 L CNN
-F 2 "Capacitor_SMD:C_0603_1608Metric" H 8388 4550 50  0001 C CNN
+F 2 "Capacitor_SMD:C_0402_1005Metric" H 8388 4550 50  0001 C CNN
 F 3 "~" H 8350 4700 50  0001 C CNN
 	1    8350 4700
@@
 F 0 "R5" H 5920 1296 50  0000 L CNN
 F 1 "270R" H 5920 1205 50  0000 L CNN
-F 2 "Resistor_SMD:R_0603_1608Metric" V 5780 1250 50  0001 C CNN
+F 2 "Resistor_SMD:R_0402_1005Metric" V 5780 1250 50  0001 C CNN
 F 3 "~" H 5850 1250 50  0001 C CNN
 	1    5850 1250
@@
 F 0 "C23" H 8965 4646 50  0000 L CNN
 F 1 "10nF" H 8965 4555 50  0000 L CNN
-F 2 "Capacitor_SMD:C_0603_1608Metric" H 8888 4450 50  0001 C CNN
+F 2 "Capacitor_SMD:C_0402_1005Metric" H 8888 4450 50  0001 C CNN
 F 3 "~" H 8850 4600 50  0001 C CNN
 	1    8850 4600
@@
 F 0 "C18" H 7015 2846 50  0000 L CNN
 F 1 "22pF" H 7015 2755 50  0000 L CNN
-F 2 "Capacitor_SMD:C_0603_1608Metric" H 6938 2650 50  0001 C CNN
+F 2 "Capacitor_SMD:C_0402_1005Metric" H 6938 2650 50  0001 C CNN
 F 3 "~" H 6900 2800 50  0001 C CNN
 	1    6900 2800
@@
 F 0 "R4" H 5470 1296 50  0000 L CNN
 F 1 "560R" H 5470 1205 50  0000 L CNN
-F 2 "Resistor_SMD:R_0603_1608Metric" V 5330 1250 50  0001 C CNN
+F 2 "Resistor_SMD:R_0402_1005Metric" V 5330 1250 50  0001 C CNN
 F 3 "~" H 5400 1250 50  0001 C CNN
 	1    5400 1250
@@
 F 0 "C16" H 5965 1696 50  0000 L CNN
 F 1 "15nF" H 5965 1605 50  0000 L CNN
-F 2 "Capacitor_SMD:C_0603_1608Metric" H 5888 1500 50  0001 C CNN
+F 2 "Capacitor_SMD:C_0402_1005Metric" H 5888 1500 50  0001 C CNN
 F 3 "~" H 5850 1650 50  0001 C CNN
 	1    5850 1650
@@
 F 0 "C14" H 5515 1696 50  0000 L CNN
 F 1 "470pF" H 5515 1605 50  0000 L CNN
-F 2 "Capacitor_SMD:C_0603_1608Metric" H 5438 1500 50  0001 C CNN
+F 2 "Capacitor_SMD:C_0402_1005Metric" H 5438 1500 50  0001 C CNN
 F 3 "~" H 5400 1650 50  0001 C CNN
 	1    5400 1650
@@
 F 0 "C17" H 6415 1446 50  0000 L CNN
 F 1 "1nF" H 6415 1355 50  0000 L CNN
-F 2 "Capacitor_SMD:C_0603_1608Metric" H 6338 1250 50  0001 C CNN
+F 2 "Capacitor_SMD:C_0402_1005Metric" H 6338 1250 50  0001 C CNN
 F 3 "~" H 6300 1400 50  0001 C CNN
 	1    6300 1400
@@
 F 0 "C20" H 7835 3546 50  0000 R CNN
 F 1 "100nF" H 7835 3455 50  0000 R CNN
-F 2 "Capacitor_SMD:C_0603_1608Metric" H 7988 3350 50  0001 C CNN
+F 2 "Capacitor_SMD:C_0402_1005Metric" H 7988 3350 50  0001 C CNN
 F 3 "~" H 7950 3500 50  0001 C CNN
 	1    7950 3500
@@
 F 0 "C15" V 5548 3050 50  0000 C CNN
 F 1 "22nF" V 5639 3050 50  0000 C CNN
-F 2 "Capacitor_SMD:C_0603_1608Metric" H 5838 2900 50  0001 C CNN
+F 2 "Capacitor_SMD:C_0402_1005Metric" H 5838 2900 50  0001 C CNN
 F 3 "~" H 5800 3050 50  0001 C CNN
 	1    5800 3050
@@
 F 0 "C11" H 4765 3996 50  0000 L CNN
 F 1 "10nF" H 4765 3905 50  0000 L CNN
-F 2 "Capacitor_SMD:C_0603_1608Metric" H 4688 3800 50  0001 C CNN
+F 2 "Capacitor_SMD:C_0402_1005Metric" H 4688 3800 50  0001 C CNN
 F 3 "~" H 4650 3950 50  0001 C CNN
 	1    4650 3950
@@
 F 0 "R6" V 7700 4250 50  0000 C CNN
 F 1 "1K" V 7750 4400 50  0000 C CNN
-F 2 "Resistor_SMD:R_0603_1608Metric" V 7630 4250 50  0001 C CNN
+F 2 "Resistor_SMD:R_0402_1005Metric" V 7630 4250 50  0001 C CNN
 F 3 "~" H 7700 4250 50  0001 C CNN
 	1    7700 4250
@@
 F 0 "R7" V 7850 4150 50  0000 C CNN
 F 1 "1K" V 7900 4300 50  0000 C CNN
-F 2 "Resistor_SMD:R_0603_1608Metric" V 7780 4150 50  0001 C CNN
+F 2 "Resistor_SMD:R_0402_1005Metric" V 7780 4150 50  0001 C CNN
 F 3 "~" H 7850 4150 50  0001 C CNN
 	1    7850 4150
@@
 F 0 "R8" V 7950 4050 50  0000 C CNN
 F 1 "1K" V 8000 4200 50  0000 C CNN
-F 2 "Resistor_SMD:R_0603_1608Metric" V 7880 4050 50  0001 C CNN
+F 2 "Resistor_SMD:R_0402_1005Metric" V 7880 4050 50  0001 C CNN
 F 3 "~" H 7950 4050 50  0001 C CNN
 	1    7950 4050
@@
 F 0 "C22" H 8615 3246 50  0000 L CNN
 F 1 "10nF" H 8615 3155 50  0000 L CNN
-F 2 "Capacitor_SMD:C_0603_1608Metric" H 8538 3050 50  0001 C CNN
+F 2 "Capacitor_SMD:C_0402_1005Metric" H 8538 3050 50  0001 C CNN
 F 3 "~" H 8500 3200 50  0001 C CNN
 	1    8500 3200
@@
 F 0 "C12" H 4636 5846 50  0000 R CNN
 F 1 "10nF" H 4636 5755 50  0000 R CNN
-F 2 "Capacitor_SMD:C_0603_1608Metric" H 4788 5650 50  0001 C CNN
+F 2 "Capacitor_SMD:C_0402_1005Metric" H 4788 5650 50  0001 C CNN
 F 3 "~" H 4750 5800 50  0001 C CNN
 	1    4750 5800
@@
 F 0 "R3" H 5020 5346 50  0000 L CNN
 F 1 "3K6" H 5020 5255 50  0000 L CNN
-F 2 "Resistor_SMD:R_0603_1608Metric" V 4880 5300 50  0001 C CNN
+F 2 "Resistor_SMD:R_0402_1005Metric" V 4880 5300 50  0001 C CNN
 F 3 "~" H 4950 5300 50  0001 C CNN
 	1    4950 5300
@@
 F 0 "C13" H 5315 5846 50  0000 L CNN
 F 1 "100nF" H 5315 5755 50  0000 L CNN
-F 2 "Capacitor_SMD:C_0603_1608Metric" H 5238 5650 50  0001 C CNN
+F 2 "Capacitor_SMD:C_0402_1005Metric" H 5238 5650 50  0001 C CNN
 F 3 "~" H 5200 5800 50  0001 C CNN
 	1    5200 5800
@@
 F 0 "R1" H 4220 5196 50  0000 L CNN
 F 1 "1K1" H 4220 5105 50  0000 L CNN
-F 2 "Resistor_SMD:R_0603_1608Metric" V 4080 5150 50  0001 C CNN
+F 2 "Resistor_SMD:R_0402_1005Metric" V 4080 5150 50  0001 C CNN
 F 3 "~" H 4150 5150 50  0001 C CNN
 	1    4150 5150
@@
 F 0 "C9" H 3665 5196 50  0000 L CNN
 F 1 "11pF" H 3665 5105 50  0000 L CNN
-F 2 "Capacitor_SMD:C_0603_1608Metric" H 3588 5000 50  0001 C CNN
+F 2 "Capacitor_SMD:C_0402_1005Metric" H 3588 5000 50  0001 C CNN
 F 3 "~" H 3550 5150 50  0001 C CNN
 	1    3550 5150
@@
 F 0 "C7" V 3300 4400 50  0000 C CNN
 F 1 "11pF" V 3400 4400 50  0000 C CNN
-F 2 "Capacitor_SMD:C_0603_1608Metric" H 3288 4400 50  0001 C CNN
+F 2 "Capacitor_SMD:C_0402_1005Metric" H 3288 4400 50  0001 C CNN
 F 3 "~" H 3250 4550 50  0001 C CNN
 	1    3250 4550
@@
 F 0 "C36" V 3750 4200 50  0000 C CNN
 F 1 "11pF" V 3850 4200 50  0000 C CNN
-F 2 "Capacitor_SMD:C_0603_1608Metric" H 3738 4200 50  0001 C CNN
+F 2 "Capacitor_SMD:C_0402_1005Metric" H 3738 4200 50  0001 C CNN
 F 3 "~" H 3700 4350 50  0001 C CNN
 	1    3700 4350
@@
 F 0 "C35" H 2665 4846 50  0000 L CNN
 F 1 "C" H 2665 4755 50  0000 L CNN
-F 2 "Capacitor_SMD:C_0603_1608Metric" H 2588 4650 50  0001 C CNN
+F 2 "Capacitor_SMD:C_0402_1005Metric" H 2588 4650 50  0001 C CNN
 F 3 "~" H 2550 4800 50  0001 C CNN
 	1    2550 4800
@@
 F 0 "C34" H 2165 4846 50  0000 L CNN
 F 1 "6.8pF" H 2165 4755 50  0000 L CNN
-F 2 "Capacitor_SMD:C_0603_1608Metric" H 2088 4650 50  0001 C CNN
+F 2 "Capacitor_SMD:C_0402_1005Metric" H 2088 4650 50  0001 C CNN
 F 3 "~" H 2050 4800 50  0001 C CNN
 	1    2050 4800
@@
 F 0 "C4" H 1665 4846 50  0000 L CNN
 F 1 "C" H 1665 4755 50  0000 L CNN
-F 2 "Capacitor_SMD:C_0603_1608Metric" H 1588 4650 50  0001 C CNN
+F 2 "Capacitor_SMD:C_0402_1005Metric" H 1588 4650 50  0001 C CNN
 F 3 "~" H 1550 4800 50  0001 C CNN
 	1    1550 4800
