File: M.2 Type 2242-XX-B/M.2 Type 2242-XX-B.sch (KiCad schematic (older format))
At the start: 2 parts, among them J1 ANT1, J2 ANT2

Commit message: Schematic updated to STM32F103
Changed lines of the file:
@@
 F18 "USB_D-" B L 4900 3550 50
 F19 "LED1" O L 4900 3700 50
-F20 "UART4_TX" O L 4900 4150 50
-F21 "SOFT_RESET" I L 4900 4300 50
+F20 "SOFT_RESET" I L 4900 4300 50
+F21 "UART_TX" O L 4900 4150 50
 $EndSheet
 $Sheet

Commit message: Almost everything placed
Parts:
- renumbered J1 to J101, J2 to J102
Changed lines of the file:
@@
 $EndDescr
 $Comp
-L Connector:Conn_Coaxial J1
+L Connector:Conn_Coaxial J101
 U 1 1 5DA1DA4F
 P 8550 3650
-F 0 "J1" H 8650 3625 50  0000 L CNN
+F 0 "J101" H 8650 3625 50  0000 L CNN
 F 1 "ANT1" H 8650 3534 50  0000 L CNN
 F 2 "Connector_Coaxial:U.FL_Hirose_U.FL-R-SMT-1_Vertical" H 8550 3650 50  0001 C CNN
@@
 $EndComp
 $Comp
-L Connector:Conn_Coaxial J2
+L Connector:Conn_Coaxial J102
 U 1 1 5DA1DFAE
 P 8550 4250
-F 0 "J2" H 8650 4225 50  0000 L CNN
+F 0 "J102" H 8650 4225 50  0000 L CNN
 F 1 "ANT2" H 8650 4134 50  0000 L CNN
 F 2 "Connector_Coaxial:U.FL_Hirose_U.FL-R-SMT-1_Vertical" H 8550 4250 50  0001 C CNN
@@
 	8350 4250 8200 4250
 $Comp
-L power:GND #PWR0107
+L power:GND #PWR0101
 U 1 1 5DC3C07A
 P 8550 3850
-F 0 "#PWR0107" H 8550 3600 50  0001 C CNN
+F 0 "#PWR0101" H 8550 3600 50  0001 C CNN
 F 1 "GND" H 8555 3677 50  0000 C CNN
 F 2 "" H 8550 3850 50  0001 C CNN
@@
 $EndComp
 $Comp
-L power:GND #PWR0108
+L power:GND #PWR0102
 U 1 1 5DC3C39B
 P 8550 4450
-F 0 "#PWR0108" H 8550 4200 50  0001 C CNN
+F 0 "#PWR0102" H 8550 4200 50  0001 C CNN
 F 1 "GND" H 8555 4277 50  0000 C CNN
 F 2 "" H 8550 4450 50  0001 C CNN

Commit message: Update clearance rules for M.2 fingers
Parts:
- J101: value ANT1 -> A
- J102: value ANT2 -> B
Changed lines of the file:
@@
 P 8550 3650
 F 0 "J101" H 8650 3625 50  0000 L CNN
-F 1 "ANT1" H 8650 3534 50  0000 L CNN
+F 1 "A" H 8650 3534 50  0000 L CNN
 F 2 "Connector_Coaxial:U.FL_Hirose_U.FL-R-SMT-1_Vertical" H 8550 3650 50  0001 C CNN
 F 3 " ~" H 8550 3650 50  0001 C CNN
@@
 P 8550 4250
 F 0 "J102" H 8650 4225 50  0000 L CNN
-F 1 "ANT2" H 8650 4134 50  0000 L CNN
+F 1 "B" H 8650 4134 50  0000 L CNN
 F 2 "Connector_Coaxial:U.FL_Hirose_U.FL-R-SMT-1_Vertical" H 8550 4250 50  0001 C CNN
 F 3 " ~" H 8550 4250 50  0001 C CNN
